Commit message: Update robot model

File: swervebot_description/urdf/mobile_base.xacro (robot description, xacro)
@@ -105,5 +105,5 @@
         <parent link="front_left_caster_link" />
         <child link="front_left_wheel_link" />
-        <origin xyz="0 ${caster_width / 2 + wheel_length / 2} ${-wheel_radius / 2}" rpy="0 0 0"/>
+        <origin xyz="0 0 ${-wheel_radius / 2}" rpy="0 0 0"/>
         <axis xyz="0 1 0" />
     </joint>
@@ -111,5 +111,5 @@
         <parent link="front_right_caster_link" />
         <child link="front_right_wheel_link" />
-        <origin xyz="0 ${-caster_width / 2 - wheel_length / 2} ${-wheel_radius / 2}" rpy="0 0 0"/>
+        <origin xyz="0 0 ${-wheel_radius / 2}" rpy="0 0 0"/>
         <axis xyz="0 1 0" />
     </joint>
@@ -117,5 +117,5 @@
         <parent link="back_left_caster_link" />
         <child link="back_left_wheel_link" />
-        <origin xyz="0 ${caster_width / 2 + wheel_length / 2} ${-wheel_radius / 2}" rpy="0 0 0"/>
+        <origin xyz="0 0 ${-wheel_radius / 2}" rpy="0 0 0"/>
         <axis xyz="0 1 0" />
     </joint>
@@ -123,5 +123,5 @@
         <parent link="back_right_caster_link" />
         <child link="back_right_wheel_link" />
-        <origin xyz="0 ${-caster_width / 2 - wheel_length / 2} ${-wheel_radius / 2}" rpy="0 0 0"/>
+        <origin xyz="0 0 ${-wheel_radius / 2}" rpy="0 0 0"/>
         <axis xyz="0 1 0" />
     </joint>

File: swervebot_description/urdf/swerve_robot_ros2_control.xacro (robot description, xacro)
@@ -9,6 +9,6 @@
     <joint name="base_frontleft_caster_joint">
       <command_interface name="position">
-        <param name="min">-3.14159</param>
-        <param name="max"> 3.14159</param>
+        <param name="min">-3.1416</param>
+        <param name="max"> 3.1416</param>
       </command_interface>
       <state_interface name="position">
@@ -19,6 +19,6 @@
     <joint name="base_frontright_caster_joint">
       <command_interface name="position">
-        <param name="min">-3.14159</param>
-        <param name="max"> 3.14159</param>
+        <param name="min">-3.1416</param>
+        <param name="max"> 3.1416</param>
       </command_interface>
       <state_interface name="position">
@@ -29,6 +29,6 @@
     <joint name="base_backleft_caster_joint">
       <command_interface name="position">
-        <param name="min">-3.14159</param>
-        <param name="max"> 3.14159</param>
+        <param name="min">-3.1416</param>
+        <param name="max"> 3.1416</param>
       </command_interface>
       <state_interface name="position">
@@ -39,6 +39,6 @@
     <joint name="base_backright_caster_joint">
       <command_interface name="position">
-        <param name="min">-3.14159</param>
-        <param name="max"> 3.14159</param>
+        <param name="min">-3.1416</param>
+        <param name="max"> 3.1416</param>
       </command_interface>
       <state_interface name="position">
